File: minimote.sch (EAGLE design)
At the start: 41 parts, among them IC1 ATTINY441/841-SSU, J1 AVR_SPI_PROG_3X2PTH, T1 2N3904

Commit message: moved parts around
Parts:
- renumbered U$3 to U$13
Connections:
- new net N$123: D4.C, D5.A, D6.A, R1.2
- new net N$124: D1.C, D3.A, D4.A, D5.C, R4.2
- new net N$125: D1.A, D3.C, D6.C, R7.2
- net LED1: no longer D1.A, D3.C, D6.C, R7.2
- net LED2: no longer D1.C, D3.A, D4.A, D5.C, R4.2
- net LED3: no longer D4.C, D5.A, D6.A, R1.2

Commit message: changed 3904 to smt component
Parts:
- T1: value 2N3904 -> (none); device transistor:2N3904 -> transistor:MMBT3904LT1-NPN-SOT23-BEC
Changed lines of the file:
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@@
 <part name="GND1" library="supply1" library_urn="urn:adsk.eagle:library:371" deviceset="GND" device=""/>
 <part name="IR" library="SparkFun-LED" deviceset="LED" device="3MM"/>
-<part name="T1" library="transistor" library_urn="urn:adsk.eagle:library:402" deviceset="2N3904" device="" package3d_urn="urn:adsk.eagle:package:29893/2"/>
 <part name="GND2" library="supply1" library_urn="urn:adsk.eagle:library:371" deviceset="GND" device=""/>
 <part name="GND3" library="supply1" library_urn="urn:adsk.eagle:library:371" deviceset="GND" device=""/>
@@
 <part name="U$13" library="minimote" deviceset="EDGEUSB" device=""/>
 <part name="U$4" library="minimote" deviceset="AZ23C3V6" device=""/>
+<part name="T1" library="transistor" library_urn="urn:adsk.eagle:library:402" deviceset="*-NPN-" device="SOT23-BEC" package3d_urn="urn:adsk.eagle:package:29919/2" technology="MMBT3904LT1"/>
 </parts>
 <sheets>
@@
 <instance part="GND1" gate="1" x="-5.08" y="7.62"/>
 <instance part="IR" gate="G$1" x="129.54" y="-10.16"/>
-<instance part="T1" gate="G1" x="127" y="-22.86"/>
 <instance part="GND2" gate="1" x="-17.78" y="12.7"/>
 <instance part="GND3" gate="1" x="58.42" y="-17.78"/>
@@
 <instance part="U$13" gate="G$1" x="116.84" y="73.66"/>
 <instance part="U$4" gate="G$1" x="81.28" y="68.58" rot="R180"/>
+<instance part="T1" gate="G$1" x="127" y="-22.86"/>
 </instances>
 <busses>
@@
 <label x="53.34" y="-15.24" size="1.778" layer="95"/>
 <pinref part="J1" gate="G$1" pin="6"/>
-</segment>
-<segment>
-<pinref part="T1" gate="G1" pin="E"/>
-<pinref part="GND4" gate="1" pin="GND"/>
 </segment>
 <segment>
@@
 <pinref part="U$13" gate="G$1" pin="GND"/>
 <pinref part="U$4" gate="G$1" pin="AA"/>
+</segment>
+<segment>
+<pinref part="GND4" gate="1" pin="GND"/>
+<pinref part="T1" gate="G$1" pin="E"/>
 </segment>
 </net>
@@
 <net name="N$2" class="0">
 <segment>
-<pinref part="T1" gate="G1" pin="C"/>
 <pinref part="IR" gate="G$1" pin="C"/>
 <wire x1="129.54" y1="-17.78" x2="129.54" y2="-15.24" width="0.1524" layer="91"/>
-</segment>
-</net>
-<net name="N$3" class="0">
-<segment>
-<pinref part="T1" gate="G1" pin="B"/>
-<pinref part="R3" gate="G$1" pin="2"/>
+<pinref part="T1" gate="G$1" pin="C"/>
 </segment>
 </net>
@@
 </segment>
 </net>
+<net name="N$3" class="0">
+<segment>
+<pinref part="R3" gate="G$1" pin="2"/>
+<pinref part="T1" gate="G$1" pin="B"/>
+</segment>
+</net>
